File: eagle/NinjaPCB_ver2-170831.brd (EAGLE design)
At the start: 72 x 79 mm, 81 parts, among them IC2 VNH5019/VNH3SP30-BNC, IC3 ANALOGSW_AD_SOT23-6NC, IC4 ANALOGSW_TI-SC70-5/6NC, IC5 MCP3551SNNC, IC6 NAU7802NC, J2 ATX24, J3 HEATER, J4 HEATER_TEMP, J5 PELTIER, Q2 IRF520NPBF, Q3 IRF520NPBF, U1 CJT1117-3.3-SOT223

Commit message: completed ver2-170831
Parts:
- removed CS0, IO10, IO9, MISO, MOSI, SCKL: (no value), pinhead:1X01
Connections:
- removed net N$61: ESP2.10, MISO.1
- removed net N$62: ESP2.13, MOSI.1
- removed net N$63: ESP2.14, SCKL.1
- removed net N$64: CS0.1, ESP2.9
- removed net N$72: ESP2.11, IO9.1
- removed net N$73: ESP2.12, IO10.1
Routing:
- net N$63: track 11.4 -> 0.00 mm
- net N$64: track 10.2 -> 0.00 mm
- net N$61: track 8.28 -> 0.00 mm
- net N$62: track 8.08 -> 0.00 mm
- net N$72: track 4.93 -> 0.00 mm
- net N$73: track 4.71 -> 0.00 mm
- net GND: vias 69 -> 81
Other:
- board text added: "ESP-WROOM-02"
- board text removed: "ESP -WROOM-02"
Changed lines of the file:
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@@
 <text x="66.04" y="-70.0278" size="1.27" layer="22" rot="MR90">RX</text>
 <text x="66.04" y="-60.5536" size="1.27" layer="22" rot="MR90">GND</text>
-<text x="64.9986" y="-52.959" size="1.27" layer="22" rot="MR0">ESP
--WROOM-02</text>
-<text x="51.4096" y="-49.3014" size="1.27" layer="21" rot="SR0">ESP-12F</text>
+<text x="63.4492" y="-53.3908" size="1.27" layer="22" rot="SMR90">ESP-WROOM-02</text>
+<text x="48.4886" y="-43.1546" size="1.27" layer="21" rot="SR270">ESP-12F</text>
 <hole x="9.5" y="-76.5" drill="3.2"/>
 <text x="25.3492" y="-77.1144" size="1.778" layer="21">NinjaPCB ver2-170831</text>
@@
 <elements>
 <element name="ESP1" library="PCR-Module" package="ESP-WROOM-02-NOCREAM" value="ESP-WROOM-02NC" x="65.89" y="-46.5226" smashed="yes" rot="MR270">
-<attribute name="NAME" x="64.2484" y="-42.5646" size="1.778" layer="26" rot="MR0"/>
+<attribute name="NAME" x="48.5198" y="-49.4656" size="1.778" layer="26" rot="SMR90"/>
 </element>
 <element name="IC5" library="microchip" package="SO-08-NOCREAM" value="MCP3551SNNC" x="61.915" y="-24.6356" smashed="yes" rot="R90">
@@
 </element>
 <element name="ESP2" library="Seeed-OPL-2017-01-Sensor-camilo" package="ESP-12F" value="ESP-12F" x="58.27" y="-46.5226" smashed="yes" rot="R270">
-<attribute name="NAME" x="51.3486" y="-43.9904" size="1.778" layer="25" ratio="11"/>
+<attribute name="NAME" x="67.1346" y="-43.4238" size="1.778" layer="25" ratio="11" rot="SR270"/>
 </element>
 <element name="SJ1" library="jumper" package="SJ" value="" x="49.38" y="-33.8226" smashed="yes" rot="MR270">
@@
 <attribute name="NAME" x="58.8366" y="-6.5938" size="0.889" layer="25" ratio="11" rot="R90"/>
 <attribute name="NAME" x="59.5782" y="-3.998" size="0.635" layer="33" ratio="10" rot="R270"/>
-</element>
-<element name="IO9" library="pinhead" package="1X01" value="" x="42.0902" y="-43.7032" smashed="yes">
-<attribute name="VALUE" x="40.8202" y="-46.8782" size="1.27" layer="27"/>
-</element>
-<element name="IO10" library="pinhead" package="1X01" value="" x="42.0902" y="-46.2432" smashed="yes">
-<attribute name="VALUE" x="40.8202" y="-49.4182" size="1.27" layer="27"/>
-</element>
-<element name="MISO" library="pinhead" package="1X01" value="" x="39.5502" y="-43.7032" smashed="yes">
-<attribute name="VALUE" x="38.2802" y="-46.8782" size="1.27" layer="27"/>
-</element>
-<element name="MOSI" library="pinhead" package="1X01" value="" x="39.5502" y="-46.2432" smashed="yes">
-<attribute name="VALUE" x="38.2802" y="-49.4182" size="1.27" layer="27"/>
-</element>
-<element name="SCKL" library="pinhead" package="1X01" value="" x="37.0102" y="-46.2432" smashed="yes">
-<attribute name="VALUE" x="35.7402" y="-49.4182" size="1.27" layer="27"/>
-</element>
-<element name="CS0" library="pinhead" package="1X01" value="" x="37.0102" y="-43.7032" smashed="yes">
-<attribute name="VALUE" x="35.7402" y="-46.8782" size="1.27" layer="27"/>
 </element>
 <element name="R10" library="Seeed-Resistor" package="R0603" value="3K" x="41.4782" y="-17.8054" smashed="yes">
@@
 <wire x1="4.6863" y1="-11.2649" x2="4.6863" y2="-10.7037" width="2.54" layer="1"/>
 <wire x1="4.6863" y1="-10.7037" x2="5.79" y2="-9.6" width="2.54" layer="1"/>
+<via x="36.1696" y="-43.2562" extent="1-16" drill="0.6"/>
+<via x="38.2016" y="-43.2562" extent="1-16" drill="0.6"/>
+<via x="40.2336" y="-43.2562" extent="1-16" drill="0.6"/>
+<via x="42.2656" y="-43.2562" extent="1-16" drill="0.6"/>
+<via x="36.1696" y="-45.2882" extent="1-16" drill="0.6"/>
+<via x="38.2016" y="-45.2882" extent="1-16" drill="0.6"/>
+<via x="40.2336" y="-45.2882" extent="1-16" drill="0.6"/>
+<via x="42.2656" y="-45.2882" extent="1-16" drill="0.6"/>
+<via x="36.1696" y="-47.3202" extent="1-16" drill="0.6"/>
+<via x="38.2016" y="-47.3202" extent="1-16" drill="0.6"/>
+<via x="40.2336" y="-47.3202" extent="1-16" drill="0.6"/>
+<via x="42.2656" y="-47.3202" extent="1-16" drill="0.6"/>
 </signal>
 <signal name="3V3">
@@
 <wire x1="61.8768" y1="-35.8546" x2="62.08" y2="-35.8546" width="0.3048" layer="1"/>
 </signal>
-<signal name="N$61">
-<contactref element="MISO" pad="1"/>
-<contactref element="ESP2" pad="10"/>
-<wire x1="46.27" y1="-43.5226" x2="45.8512" y2="-43.1038" width="0.3048" layer="1"/>
-<wire x1="39.5502" y1="-43.7032" x2="40.1422" y2="-43.7032" width="0.3048" layer="1"/>
-<wire x1="40.1422" y1="-43.7032" x2="41.402" y2="-42.4434" width="0.3048" layer="1"/>
-<wire x1="41.402" y1="-42.4434" x2="43.561" y2="-42.4434" width="0.3048" layer="1"/>
-<wire x1="43.561" y1="-42.4434" x2="44.6402" y2="-43.5226" width="0.3048" layer="1"/>
-<wire x1="44.6402" y1="-43.5226" x2="46.27" y2="-43.5226" width="0.3048" layer="1"/>
-</signal>
-<signal name="N$62">
-<contactref element="MOSI" pad="1"/>
-<contactref element="ESP2" pad="13"/>
-<wire x1="39.5502" y1="-46.2432" x2="40.071" y2="-46.2432" width="0.3048" layer="1"/>
-<wire x1="40.071" y1="-46.2432" x2="43.3504" y2="-49.5226" width="0.3048" layer="1"/>
-<wire x1="43.3504" y1="-49.5226" x2="46.27" y2="-49.5226" width="0.3048" layer="1"/>
-</signal>
-<signal name="N$63">
-<contactref element="SCKL" pad="1"/>
-<contactref element="ESP2" pad="14"/>
-<wire x1="37.0102" y1="-46.2432" x2="38.3412" y2="-47.5742" width="0.3048" layer="1"/>
-<wire x1="38.3412" y1="-47.5742" x2="40.3098" y2="-47.5742" width="0.3048" layer="1"/>
-<wire x1="40.3098" y1="-47.5742" x2="44.2582" y2="-51.5226" width="0.3048" layer="1"/>
-<wire x1="44.2582" y1="-51.5226" x2="46.27" y2="-51.5226" width="0.3048" layer="1"/>
-</signal>
-<signal name="N$64">
-<contactref element="CS0" pad="1"/>
-<contactref element="ESP2" pad="9"/>
-<wire x1="46.27" y1="-41.5226" x2="40.7226" y2="-41.5226" width="0.3048" layer="1"/>
-<wire x1="39.8018" y1="-42.4434" x2="38.8112" y2="-42.4434" width="0.3048" layer="1"/>
-<wire x1="38.8112" y1="-42.4434" x2="37.5514" y2="-43.7032" width="0.3048" layer="1"/>
-<wire x1="37.5514" y1="-43.7032" x2="37.0102" y2="-43.7032" width="0.3048" layer="1"/>
-<wire x1="39.8018" y1="-42.4434" x2="40.7226" y2="-41.5226" width="0.3048" layer="1"/>
-</signal>
 <signal name="N$67">
 <contactref element="ESP2" pad="6"/>
@@
 <wire x1="55.75" y1="-36.9268" x2="56.8222" y2="-35.8546" width="0.3048" layer="1"/>
 <wire x1="56.8222" y1="-35.8546" x2="57" y2="-35.8546" width="0.3048" layer="1"/>
-</signal>
-<signal name="N$72">
-<contactref element="IO9" pad="1"/>
-<contactref element="ESP2" pad="11"/>
-<wire x1="42.0902" y1="-43.7032" x2="43.9096" y2="-45.5226" width="0.3048" layer="1"/>
-<wire x1="43.9096" y1="-45.5226" x2="46.27" y2="-45.5226" width="0.3048" layer="1"/>
-</signal>
-<signal name="N$73">
-<contactref element="IO10" pad="1"/>
-<contactref element="ESP2" pad="12"/>
-<wire x1="42.0902" y1="-46.2432" x2="43.3696" y2="-47.5226" width="0.3048" layer="1"/>
-<wire x1="43.3696" y1="-47.5226" x2="46.27" y2="-47.5226" width="0.3048" layer="1"/>
 </signal>
 <signal name="IO12">
@@
 </board>
 </drawing>
-<compatibility>
-<note version="6.3" minversion="6.2.2" severity="warning">
-Since Version 6.2.2 text objects can contain more than one line,
-which will not be processed correctly with this version.
-</note>
-</compatibility>
 </eagle>

Commit message: completed ver2-170831
Parts:
- removed R4: 1.5K or 1.8K, PCR-RCL:R0603NC
- added RD2, RH2: 30K HP, PCR-RCL:R0603NC
- RD1: value 1.5K or 1.8K -> 30K HP
- RH1: value 15K 1/10W -> 30K HP
- RL: value 30K -> 30K HP
- moved RL 2.54 mm to (54.6, -2.54)
- moved C3 0.66 mm to (60.1, -5.88), turned to 270 degrees
- turned RD1 to 0 degrees
- renumbered R11 to RD1, RH to RH1
Connections:
- net 3V3: now also RD1.2; no longer R4.2
- net GND: now also RD2.1; no longer RD1.1
- net N$27: now also RH2.1
- net N$91: now also RD1.1, RD2.2; no longer R4.1, RD1.2
- net WELL_TEMP: now also RH2.2
Routing:
- net N$27: track 14.2 -> 16.7 mm
- net 3V3: track 239.5 -> 242.0 mm
- net N$91: track 20.2 -> 18.1 mm
- net GND: track 700.9 -> 701.9 mm
Other:
- board text added: "BLACK"
- board text added: "High Precision"
- board text added: "RED"

Commit message: completed ver2-170831
Parts:
- moved IC3 4.17 mm to (54.4, -10.5)
- moved IC4 4.17 mm to (49.3, -10.5)
Routing:
- net 3V3: track 242.0 -> 236.1 mm
- net HIGH_TEMP: track 123.2 -> 118.7 mm
- net N$27: track 16.7 -> 20.2 mm
