File: eagle/NinjaPCB-2x2-MooMoo-power_ver2.0.brd (EAGLE design)
At the start: 57 x 57 mm, 32 parts, among them J3 HEATER, Q1 S8550, Q2 IRF520NPBF, Q4 S8550, Q5 IRF520NPBF, Q6 S8550, Q7 S8550, Q8 S8550, U1 CJT1117-3.3-SOT223

Commit message: change values of MOSFET G-S reg
Parts:
- R13, R20: value 10K 1/10W -> 100K 1/10W
Changed lines of the file:
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@@
 <attribute name="MPN" value="RC0603JR-0710KL" x="26" y="2" size="1.778" layer="27" display="off"/>
 </element>
-<element name="R13" library="Seeed-Resistor" package="R0603" value="10K 1/10W" x="-28.61" y="68.04">
-<attribute name="MPN" value="RC0603JR-0710KL" x="26" y="2" size="1.778" layer="27" display="off"/>
+<element name="R13" library="Seeed-Resistor" package="R0603" value="100K 1/10W" x="-28.61" y="68.04">
+<attribute name="MPN" value="RC0603JR-07100KL" x="26" y="2" size="1.778" layer="27" display="off"/>
 </element>
 <element name="Q5" library="Seeed-Transistor" package="TO-220" value="IRF520NPBF" x="30.03" y="19.23" rot="R90"/>
@@
 <attribute name="MPN" value="RC0603JR-0710KL" x="26" y="2" size="1.778" layer="27" display="off"/>
 </element>
-<element name="R20" library="Seeed-Resistor" package="R0603" value="10K 1/10W" x="0.6" y="75.66">
-<attribute name="MPN" value="RC0603JR-0710KL" x="26" y="2" size="1.778" layer="27" display="off"/>
+<element name="R20" library="Seeed-Resistor" package="R0603" value="100K 1/10W" x="0.6" y="75.66">
+<attribute name="MPN" value="RC0603JR-07100KL" x="26" y="2" size="1.778" layer="27" display="off"/>
 </element>
 <element name="RELAY" library="PCR-Switch" package="NEC-EP2" value="NEC-RELAY2EP2" x="9.37" y="25.48" rot="R90"/>
