File: eagle/NinjaPCB_ver2.1.brd (EAGLE design)
At the start: 70 x 86 mm, 60 parts, among them IC3 ANALOGSW_AD_SOT23-6, IC6 NAU7802, J2 ATX24, J3 HEATER, J4 HEATER_TEMP, Q1 S8550, Q2 IRF520NPBF, Q3 IRF520NPBF, Q4 S8550, Q5 IRF520NPBF, Q6 S8550, Q7 S8550, Q8 S8550, U1 CJT1117-3.3-SOT223

Commit message: use easier parts. add notes to design
Parts:
- R13, R17, R20: value 100K 1/10W -> 10K 1/10W
- R14: value 2K -> 15KHP

Commit message: change values of MOSFET G-S reg
Parts:
- R13, R17, R20: value 10K 1/10W -> 100K 1/10W
