File: eagle/NinjaPCB_ver2.1.brd (EAGLE design)
At the start: 79 x 73 mm, 72 parts, among them IC1 ANALOGSW_AD_SOT23-6, IC2 NAU7802, Q1 IRLB3813PBF, Q2 CJ2302, Q3 CJ2302, Q4 S9013, Q5 S9013, Q6 S9013

Commit message: ver2.1 finished
Parts:
- moved U$7 6.97 mm to (1.17, 67.8)
Routing:
- net GND: track 917.3 -> 917.8 mm
Changed lines of the file:
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@@
 <setting verticaltext="up"/>
 </settings>
-<grid distance="1" unitdist="mm" unit="mm" style="lines" multiple="1" display="yes" altdistance="0.025" altunitdist="inch" altunit="inch"/>
+<grid distance="1" unitdist="mil" unit="mil" style="lines" multiple="1" display="yes" altdistance="0.025" altunitdist="inch" altunit="inch"/>
 <layers>
 <layer number="1" name="Top" color="4" fill="1" visible="yes" active="yes"/>
@@
 <element name="Q1" library="transistor-power" package="TO220BV" value="IRLB3813PBF" x="13.3038" y="52.0942" smashed="yes" rot="R270"/>
 <element name="ESP-WROOM-02-BREAK" library="PCR-Module" package="ESP-WROOM-02-BREAK-NODETAIL" value="ESP-WROOM-02-BREAKND" x="65.8044" y="30.539" smashed="yes" rot="R270"/>
-<element name="U$7" library="adafruit" package="FIDUCIAL_1MM" value="FIDUCIAL" x="6.8072" y="71.9328" smashed="yes"/>
+<element name="U$7" library="adafruit" package="FIDUCIAL_1MM" value="FIDUCIAL" x="1.1684" y="67.8434" smashed="yes"/>
 <element name="U$8" library="adafruit" package="FIDUCIAL_1MM" value="FIDUCIAL" x="58.166" y="21.59" smashed="yes" rot="R270"/>
 <element name="U$9" library="adafruit" package="FIDUCIAL_1MM" value="FIDUCIAL" x="53.467" y="46.609" smashed="yes" rot="R270"/>
@@
 <via x="61.7982" y="5.8674" extent="1-16" drill="0.6" shape="square"/>
 <via x="16.4592" y="32.7152" extent="1-16" drill="0.6" shape="square"/>
-<via x="1.7272" y="67.1068" extent="1-16" drill="0.6" shape="square"/>
+<via x="1.2446" y="66.1416" extent="1-16" drill="0.6" shape="square"/>
 <via x="1.8288" y="49.3268" extent="1-16" drill="0.6" shape="square"/>
 <via x="7.112" y="43.688" extent="1-16" drill="0.6" shape="square"/>
@@
 <wire x1="67.9704" y1="10.8204" x2="66.2178" y2="10.8204" width="0.4064" layer="1"/>
 <wire x1="66.2178" y1="10.8204" x2="63.8302" y2="13.208" width="0.4064" layer="1"/>
-<wire x1="1.7272" y1="67.1068" x2="7.493" y2="67.1068" width="0.4064" layer="16"/>
+<wire x1="1.2446" y1="66.1416" x2="7.493" y2="67.1068" width="0.4064" layer="16"/>
 <wire x1="7.493" y1="67.1068" x2="9.1948" y2="65.405" width="0.4064" layer="16"/>
 <wire x1="37.6682" y1="24.4094" x2="42.2402" y2="24.4094" width="0.4064" layer="16"/>

Commit message: minor update of silk
Parts:
- RT: value 5K HP -> 4.99K HP
- moved U$6 1.00 mm to (39.5, 44.7)
- renumbered ESP-12 to ESP1, ESP-WROOM-02 to ESP2, ESP-WROOM-02-BREAK to ESP3
Other:
- board text added: "ESP1 ESP-12"
- board text added: "ESP2 ESP-WROOM-02"
- board text added: "center"
- board text added: "lid"
- board text added: "pipe"
- board text added: "well"
- board text removed: "ESP-12"
- board text removed: "ESP-WROOM-02"

Commit message: minor update for layout
Routing:
- net 12V: track 195.4 -> 234.3 mm

Commit message: minor update for layout
Routing:
- net 12V: track 234.3 -> 248.3 mm
Changed lines of the file:
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@@
 <wire x1="28.372" y1="27.8386" x2="28.3591" y2="27.8386" width="0.254" layer="1"/>
 <wire x1="28.3591" y1="27.8386" x2="28.3591" y2="27.8511" width="0.254" layer="1"/>
+<wire x1="19.2532" y1="21.3868" x2="19.2532" y2="15.2146" width="2.54" layer="1"/>
+<wire x1="19.2532" y1="15.2146" x2="21.8948" y2="12.573" width="2.54" layer="1"/>
+<wire x1="19.2532" y1="15.2146" x2="20.3962" y2="15.2146" width="0.254" layer="1"/>
+<wire x1="20.3962" y1="15.2146" x2="20.3962" y2="12.2936" width="0.254" layer="1"/>
 </signal>
 <signal name="N$2">

Commit message: minor update for layout
Routing:
- net 12V: track 248.3 -> 263.8 mm
Changed lines of the file:
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@@
 <wire x1="19.7358" y1="53.8226" x2="19.7358" y2="50.3428" width="2.54" layer="16"/>
 <wire x1="16.7132" y1="27.4574" x2="18.0092" y2="26.1614" width="5.08" layer="1"/>
-<wire x1="18.0092" y1="26.1614" x2="18.0092" y2="8.5726" width="5.08" layer="1"/>
+<wire x1="18.0092" y1="26.1614" x2="18.0092" y2="20.2438" width="5.08" layer="1"/>
+<wire x1="18.0092" y1="20.2438" x2="18.0092" y2="8.5726" width="5.08" layer="1"/>
 <wire x1="9.29" y1="12.1" x2="10.7282" y2="13.5382" width="5.08" layer="1"/>
 <wire x1="10.7282" y1="13.5382" x2="17.3228" y2="13.5382" width="5.08" layer="1"/>
@@
 <wire x1="19.2532" y1="15.2146" x2="20.3962" y2="15.2146" width="0.254" layer="1"/>
 <wire x1="20.3962" y1="15.2146" x2="20.3962" y2="12.2936" width="0.254" layer="1"/>
+<wire x1="17.1958" y1="23.2664" x2="17.1958" y2="20.0152" width="2.54" layer="1"/>
+<wire x1="17.1958" y1="20.0152" x2="12.065" y2="14.8844" width="2.54" layer="1"/>
+<wire x1="12.065" y1="14.8844" x2="14.5542" y2="14.8844" width="2.54" layer="1"/>
+<wire x1="14.5542" y1="14.8844" x2="15.5956" y2="15.9258" width="2.54" layer="1"/>
+<wire x1="17.1958" y1="20.0152" x2="18.0092" y2="20.0152" width="0.254" layer="1"/>
+<wire x1="18.0092" y1="20.0152" x2="18.0092" y2="20.2438" width="0.254" layer="1"/>
 </signal>
 <signal name="N$2">
