File: eagle/NinjaPCB-4x4-NinNin_ver2.0.sch (EAGLE design)
At the start: 71 parts, among them IC3 ANALOGSW_AD_SOT23-6, IC6 NAU7802, J2 ATX24NH, J3 HEATER, J4 HEATER_TEMP, Q1 CJ2302, Q10 S9013, Q11 S9013, Q2 IRLB3813PBF, Q4 CJ2302, Q9 S9013, U1 CJT1117-3.3-SOT223

Commit message: ready to order
Parts:
- removed C7: CAP_SMDAL_1000UF_25V, Seeed-OPL-2017-01-Capacitor-akita:CAP_SMDAL_1000UF_25V
- removed ESP3: ESP-WROOM-02-BREAK, PCR-Module:ESP-WROOM-02-BREAK
- removed Q9: S9013, Seeed-Transistor:SMD-TRANSISTORS-NPN-25V-500MA-S9013(SOT-23)
- removed R19, R20: 10K 1/10W, Seeed-Resistor:SMD-RES-10K-5%-1/10W(0603)
- added C1: 100nf, Seeed-Capacitor:CERAMIC-100NF-50V-10%-X7R(0603)
- added ESP-WROOM-02-BREAK: ESP-WROOM-02-BREAKND, PCR-Module:ESP-WROOM-02-BREAKND
- added Q3: CJ2302, Seeed-Transistor:SMD-MOSFET-N-CH-20V-2.1A-CJ2302(SOT-23)
- added R6, R8: 10K 1/10W, Seeed-Resistor:SMD-RES-10K-5%-1/10W(0603)
- C3: value 100nf -> CAP_SMDAL_1000UF_25V; device Seeed-Capacitor:CERAMIC-100NF-50V-10%-X7R(0603) -> Seeed-OPL-2017-01-Capacitor-akita:CAP_SMDAL_1000UF_25V
- HEATER_POWER: value HEATER -> (none)
- HEATER_TEMP: value HEATER_TEMP -> (none)
- Q1: value CJ2302 -> IRLB3813PBF; device Seeed-Transistor:SMD-MOSFET-N-CH-20V-2.1A-CJ2302(SOT-23) -> transistor-power:IRF520
- Q2: value IRLB3813PBF -> CJ2302; device transistor-power:IRF520 -> Seeed-Transistor:SMD-MOSFET-N-CH-20V-2.1A-CJ2302(SOT-23)
- Q4: value CJ2302 -> S9013; device Seeed-Transistor:SMD-MOSFET-N-CH-20V-2.1A-CJ2302(SOT-23) -> Seeed-Transistor:SMD-TRANSISTORS-NPN-25V-500MA-S9013(SOT-23)
- R12, R17: value 10K 1/10W -> 1K 1/10W; device Seeed-Resistor:SMD-RES-10K-5%-1/10W(0603) -> Seeed-Resistor:SMD-RES-1K-5%-1/10W(0603)
- R16, R18: value 1K 1/10W -> 10K 1/10W; device Seeed-Resistor:SMD-RES-1K-5%-1/10W(0603) -> Seeed-Resistor:SMD-RES-10K-5%-1/10W(0603)
- renumbered ESP1 to ESP-12, ESP2 to ESP-WROOM-02, IC3 to IC1, IC6 to IC2, J2 to ATX, J3 to HEATER_POWER, J4 to HEATER_TEMP, JP2 to FAN, Q10 to Q5, Q11 to Q6, R21 to R10, R22 to R11, TP1 to T1, TP2 to T2, TP3 to T3, TP4 to T4, TP5 to T5, TP6 to T6, TP7 to T7, U$1 to HEATSINK, U1 to REG
Connections:
- net 12V: now also C3.P$P, R13.2; no longer C7.P$P, R19.2
- net 3V3: now also C4.+, ESP-WROOM-02-BREAK.3V3, R2.1, R3.1; no longer C2.+, ESP3.3V3, R5.1, R9.1
- net DIVIDED: now also C2.+; no longer C4.+
- net DRDY: now also ESP-WROOM-02-BREAK.IO5; no longer ESP3.IO5
- net EN: now also ESP-WROOM-02-BREAK.EN, R4.2; no longer ESP3.EN, R1.2
- net FAN: now also ESP-WROOM-02-BREAK.IO0, R17.1, R2.2; no longer ESP3.IO0, R15.1, R4.2
- net GND: now also C1.1, C3.P$M, ESP-WROOM-02-BREAK.GND13, ESP-WROOM-02-BREAK.GND18, ESP-WROOM-02-BREAK.GND9, Q3.S, Q4.E, R16.1, R18.1, R5.1, R6.1, R8.1, R9.1; no longer C3.1, C7.P$M, ESP3.GND13, ESP3.GND18, ESP3.GND9, Q4.S, Q9.E, R12.1, R13.1, R17.1, R2.1, R20.1, R3.1
- net HEATER: now also ESP-WROOM-02-BREAK.IO15/HPSICS, R15.1; no longer ESP3.IO15/HPSICS, R16.1
- net HIGH_TEMP: now also ESP-WROOM-02-BREAK.IO16, R8.2; no longer ESP3.IO16, R12.2
- net MODE: now also ESP-WROOM-02-BREAK.TOUT, R9.2; no longer ESP3.TOUT, R14.2
- net N$2: now also Q2.D; no longer Q1.D
- net N$3: now also Q1.D; no longer Q2.D
- net N$30: now also R12.2; no longer R18.2
- net N$32: now also Q2.G, R15.2; no longer Q1.G, R13.2
- net N$33: now also Q4.C; no longer Q9.C
- net N$34: now also Q4.B; no longer Q9.B
- net N$4: now also Q3.D; no longer Q4.D
- net N$5: now also Q1.G, R13.1, R14.2; no longer Q2.G, R19.1, R20.2
- net N$8: now also Q3.G, R18.2; no longer Q4.G, R15.2
- net N$92: now also C1.2; no longer C3.2
- net PEL_PWM: now also ESP-WROOM-02-BREAK.IO4, R12.1; no longer ESP3.IO4, R18.1
- net PEL_SWA: now also ESP-WROOM-02-BREAK.IO12/HSPIQ/MISO, R5.2; no longer ESP3.IO12/HSPIQ/MISO, R2.2
- net PEL_SWB: now also ESP-WROOM-02-BREAK.IO13/HSPID/MOSI, R6.2; no longer ESP3.IO13/HSPID/MOSI, R3.2
- net RESET: now also ESP-WROOM-02-BREAK.RST, R1.2; no longer ESP3.RST, R9.2
- net RXD: now also ESP-WROOM-02-BREAK.RXD; no longer ESP3.RXD
- net SCLK: now also ESP-WROOM-02-BREAK.IO14/HSPICLK; no longer ESP3.IO14/HSPICLK
- net SDIO: now also ESP-WROOM-02-BREAK.IO2, R3.2; no longer ESP3.IO2, R5.2
- net TXD: now also ESP-WROOM-02-BREAK.TXD; no longer ESP3.TXD
Other:
- moved on the sheet: C2, C4, R1, R12, R13, R14, R15, R16, R17, R18, R2, R3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
