File: eagle/NinjaPCB_ver2.0.brd (EAGLE design)
At the start: 72 x 79 mm, 76 parts, among them IC2 VNH3SP30-BNC, IC3 ANALOGSW_AD_SOT23-6NC, IC4 ANALOGSW_TI-SC70-5/6NC, IC5 MCP3551SNNC, IC6 NAU7802NC, J2 ATX24, J3 HEATER, J4 HEATER_TEMP, J5 PELTIER, Q2 IRF520NPBF, Q3 IRF520NPBF, U1 CJT1117-3.3-SOT223

Commit message: set default 4x4
Parts:
- removed C7: CAP_SMDAL_1000UF_25V, Seeed-OPL-2017-01-Capacitor-akita:CAP_SMD_AL_D125
- removed C8: 3300uF, PCR-RCL:E5-13-L30R-INV
- removed ESP1: ESP-WROOM-02NC, PCR-Module:ESP-WROOM-02-NOCREAM
- removed ESP2: ESP-12F, Seeed-OPL-2017-01-Sensor-camilo:ESP-12F
- removed IC3: ANALOGSW_AD_SOT23-6NC, PCR-IC:SOT-23-6NC
- removed IC4: ANALOGSW_TI-SC70-5/6NC, PCR-IC:SC70-6NC
- removed IC5: MCP3551SNNC, microchip:SO-08-NOCREAM
- removed IC6: NAU7802NC, PCR-IC:SOP-16NC
- removed J2: ATX24, PCR-Connector:ATX24
- removed J3: HEATER, Seeed-Connector:H2-3.5-7.0X7.0MM
- removed J4: HEATER_TEMP, Seeed-Connector:H2-3.5-7.0X7.0MM
- removed J5: PELTIER, Seeed-Connector:H2-3.5-7.0X7.0MM
- removed JP2: 22-23-2031, con-molex:22-23-2031
- removed RH1, RH2, RL: 30K HP, PCR-RCL:R0603NC
- removed SERIAL: (no value), pinhead:1X06
- removed SJ1, SJ10, SJ11, SJ12, SJ13, SJ14, SJ15, SJ16, SJ19, SJ2, SJ20, SJ21, SJ22, SJ23, SJ24, SJ25, SJ26, SJ27, SJ28, SJ29, SJ3, SJ30, SJ4, SJ5, SJ6, SJ7, SJ8, SJ9: (no value), jumper:SJ
- removed SJ17, SJ37, SJ38, SJ39, SJ40: (no value), jumper:SJ_2
- removed U1: CJT1117-3.3-SOT223, Seeed-IC:SOT-223
- removed WELLEXT1, WELLEXT2: (no value), pinhead:1X02
- added ATX: ATX24NH, PCR-Connector:ATX24
- added C1, CP1, CP2: 100nf, Seeed-Capacitor:C0603
- added C4: 22uf, Seeed-Capacitor:AVX-B
- added D1, D2: 1N4007, Seeed-Diode:DO-214AC
- added ESP-12: ESP-12F, Seeed-OPL-2017-01-Sensor-camilo:ESP-12F
- added ESP-WROOM-02: ESP-WROOM-02, PCR-Module:ESP-WROOM-02
- added ESP-WROOM-02-BREAK: ESP-WROOM-02-BREAKND, PCR-Module:ESP-WROOM-02-BREAK-NODETAIL
- added FAN: 22-23-2031, con-molex:22-23-2031
- added FAN_ON: (no value), jumper:SJ
- added HEATER_POWER, HEATER_TEMP: (no value), Seeed-Connector:H2-3.5-7.0X7.0MM
- added HEATSINK: HEAT111PB015, PCR-Connector:HEAT11PB015
- added IC1: ANALOGSW_AD_SOT23-6, PCR-IC:SOT-23-6
- added JACK: 2.1MMJACKTHM-NOOUT, adafruit:PJ-102A-NOOUT
- added PEL_BLK, PEL_RED: (no value), pinhead:1X01LONG
- added Q1: IRLB3813PBF, transistor-power:TO220BV
- added Q4, Q5, Q6: S9013, Seeed-Transistor:SOT-23
- added R11, R13, R18, R4, R7, R8: 10K 1/10W, Seeed-Resistor:R0603
- added R17: 1K 1/10W, Seeed-Resistor:R0603
- added REG: CJT1117-3.3-SOT223, Seeed-IC:SOT-223
- added RELAY: NEC-RELAY2EP2, PCR-Switch:NEC-EP2
- added RH, RL1, RL2: 15K HP, PCR-RCL:R0603
- added RT: 5K HP, Seeed-Resistor:R0603
- added SERIAL4: (no value), pinhead:1X04
- added SERIAL6: (no value), pinhead:1X06
- added T1, T2, T3, T4, T5, T6, T7: TPTP20R, testpad:TP20R
- added U$10, U$3, U$4, U$5, U$6, U$7, U$8, U$9: FIDUCIAL, adafruit:FIDUCIAL_1MM
- added U$2: (no value), PCR-Logo:TORI_0.25
- C3: value 100nf -> CAP_SMDAL_1000UF_25V; device Seeed-Capacitor:C0603 -> Seeed-OPL-2017-01-Capacitor-akita:CAP_SMD_AL_D125
- IC2: value VNH3SP30-BNC -> NAU7802; device st-microelectronics:MULTIPOWERSO-30-B-NOCREAM -> PCR-IC:SOP-16
- Q2, Q3: value IRF520NPBF -> CJ2302; device Seeed-Transistor:TO-220 -> Seeed-Transistor:SOT-23
- R1, R2, R3: value 1K 1/10W -> 10K 1/10W
- R10: value 3K -> 10K 1/10W
- R12, R15: value 10K 1/10W -> 1K 1/10W
- R14: value 2K -> 10K 1/10W
- R5, R6: value 3.3K 1/10W -> 10K 1/10W
- RD1, RD2: value 30K HP -> 15K HP; device PCR-RCL:R0603NC -> PCR-RCL:R0603
- U$1: value 2.1MMJACKTHM -> (none); device adafruit:PJ-102A -> PCR-Logo:TORI_0.25
- moved C2 139.0 mm to (42.9, 78.1), turned to 270 degrees
- moved R9 138.8 mm to (58.0, 74.9), turned to 90 degrees
- moved R12 111.4 mm to (34.0, 43.9), turned to 270 degrees
- moved R10 100.8 mm to (6.74, 76.9), turned to 90 degrees
- moved IC2 92.5 mm to (52.7, 78.8), turned to 270 degrees
- moved R3 89.0 mm to (58.0, 76.7), turned to 90 degrees
- moved IO0 87.4 mm to (57.7, 16.9), turned to 270 degrees
- moved WELL_TEMP 87.4 mm to (32.0, 83.0)
- moved MODE 87.2 mm to (50.7, 16.9), turned to 270 degrees
- moved RST 87.1 mm to (43.7, 16.9), turned to 270 degrees
- moved RD2 84.9 mm to (39.9, 80.0), turned to 270 degrees
- moved RD1 79.1 mm to (39.9, 74.7), turned to 270 degrees
- moved R5 76.2 mm to (34.0, 63.6), turned to 90 degrees
- moved R6 70.2 mm to (34.0, 60.0)
- moved Q2 69.9 mm to (26.4, 23.0), turned to 90 degrees
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Connections:
- removed net EXTADC_I2C_SCL: IC6.P$13, SJ37.3
- removed net EXTADC_I2C_SDA: IC6.P$14, SJ39.3
- removed net EXTADC_RDY: IC6.P$12, SJ40.3
- removed net I2C_WELL_TEMP: IC6.P$3, SJ17.3
- removed net INT_ADC: R10.1, R14.1, SJ30.2, SJ9.2
- removed net IO12: SJ19.1, SJ3.1, SJ38.2
- removed net IO14: SJ2.1, SJ21.1, SJ37.2
- removed net IO2: SJ27.2, SJ39.2, SJ6.1
- removed net IO5: SJ11.2, SJ29.2, SJ40.2
- removed net N$10: IC2.8, R3.2
- removed net N$11: ESP1.P$1, ESP1.P$2, SJ1.2
- removed net N$12: ESP1.P$3, SJ2.2
- removed net N$13: ESP1.P$4, SJ3.2
- removed net N$14: ESP1.P$5, SJ4.2
- removed net N$15: ESP1.P$6, SJ5.2
- removed net N$16: ESP1.P$7, SJ6.2
- removed net N$17: ESP1.P$8, SJ7.2
- removed net N$18: ESP1.P$17, SJ8.1
- removed net N$19: ESP1.P$16, SJ9.1
- removed net N$20: ESP1.P$15, SJ10.1
- removed net N$21: ESP1.P$14, SJ11.1
- removed net N$22: ESP1.P$12, SJ12.1
- removed net N$23: ESP1.P$11, SJ13.1
- removed net N$24: ESP1.P$10, SJ14.1
- removed net N$26: WELLEXT1.1, WELLEXT2.1
- removed net N$28: WELLEXT1.2, WELLEXT2.2
- removed net N$40: ESP2.1, SJ15.2
- removed net N$42: ESP2.3, ESP2.8, SJ16.2
- removed net N$43: ESP2.22, SJ24.1
- removed net N$44: ESP2.21, SJ25.1
- removed net N$45: ESP2.18, SJ26.1
- removed net N$46: ESP2.17, SJ27.1
- removed net N$47: ESP2.19, SJ28.1
- removed net N$48: ESP2.20, SJ29.1
- removed net N$49: ESP2.2, SJ30.1
- removed net N$67: ESP2.6, SJ19.2
- removed net N$68: ESP2.7, SJ20.2
- removed net N$69: ESP2.5, SJ21.2
- removed net N$70: ESP2.16, SJ22.2
- removed net N$71: ESP2.4, SJ23.2
- removed net N$9: IC2.11, R2.2
- removed net N$91: IC6.P$2, RD1.1, RD2.2
- removed net OUTA: IC2.25, IC2.30, IC2.OUTA, J5.1
- removed net OUTB: IC2.15, IC2.16, IC2.21, IC2.OUTB, J5.2
- removed net PEL_INA: R1.1, SJ38.3, SJ39.1
- removed net PEL_INB: IO0.1, IO0.4, R2.1, SJ26.2, SJ7.1
- removed net SPI_CS: IC5.7, SJ40.1
- removed net SPI_SCK: IC5.5, SJ37.1
- removed net SPI_SDO: IC5.6, SJ38.1
- removed net SPI_WELL_TEMP: IC5.2, SJ17.1
- new net DIVIDED: C2.+, IC2.P$2, IC2.P$4, RD1.1, RD2.1
- new net DRDY: ESP-12.20, ESP-WROOM-02-BREAK.P$14, ESP-WROOM-02.P$14, IC2.P$12
- new net EN: ESP-12.3, ESP-WROOM-02-BREAK.P$2, ESP-WROOM-02.P$2, R4.2
- new net HEATER_TEMP: HEATER_TEMP.2, IC2.P$5, RT.1
- new net MODE: ESP-12.2, ESP-WROOM-02-BREAK.P$16, ESP-WROOM-02.P$16, R9.2
- new net N$30: Q6.1, R12.2
- new net N$32: Q2.1, R15.2, R16.2
- new net N$33: D1.1, Q4.3, RELAY.P$3
- new net N$34: Q4.1, R10.2
- new net N$35: Q5.1, R11.1
- new net N$36: D2.1, Q5.3, RELAY.P$7
- new net PEL_SWA: ESP-12.6, ESP-WROOM-02-BREAK.P$4, ESP-WROOM-02.P$4, R10.1, R5.2
- new net PEL_SWB: ESP-12.7, ESP-WROOM-02-BREAK.P$5, ESP-WROOM-02.P$5, R11.2, R6.2
- new net SCLK: ESP-12.5, ESP-WROOM-02-BREAK.P$3, ESP-WROOM-02.P$3, IC2.P$13
- new net SDIO: ESP-12.17, ESP-WROOM-02-BREAK.P$7, ESP-WROOM-02.P$7, IC2.P$14, R3.2
- net 12V: now also ATX.10, ATX.11, C3.P$P, D1.2, D2.2, FAN.2, HEATER_POWER.1, JACK.TIP, R13.2, REG.3, RELAY.P$2, RELAY.P$4, RELAY.P$6; no longer C7.P$P, C8.+, IC2.13, IC2.23, IC2.3, IC2.VCC, J2.10, J2.11, J3.1, JP2.2, U$1.TIP, U1.3
- net 3V3: now also C4.+, CP1.1, CP2.2, ESP-12.8, ESP-WROOM-02-BREAK.P$1, ESP-WROOM-02.P$1, HEATER_TEMP.1, IC1.P$1, IC1.P$6, IC2.P$1, IC2.P$15, IC2.P$16, R1.1, R2.1, R3.1, R4.1, REG.2, REG.TER, RL1.1, SERIAL4.1, SERIAL6.4, T3.TP; no longer C2.+, IC3.P$1, IC3.P$6, IC4.P$1, IC4.P$6, IC5.1, IC5.8, IC6.P$1, IC6.P$15, IC6.P$16, J4.2, R5.1, R6.1, R9.1, RL.2, SJ1.1, SJ16.1, U1.2, U1.TER
- net FAN: now also ESP-12.18, ESP-WROOM-02-BREAK.P$8, ESP-WROOM-02.P$8, IO0.1, IO0.4, R17.1, R2.2, T5.TP; no longer R15.1, SJ20.1, SJ4.1
- net GND: now also ATX.15, ATX.17, ATX.18, ATX.19, ATX.24, ATX.3, ATX.5, ATX.7, C1.1, C3.P$M, C4.-, CP1.2, CP2.1, ESP-12.15, ESP-WROOM-02-BREAK.P$13, ESP-WROOM-02-BREAK.P$18, ESP-WROOM-02-BREAK.P$9, ESP-WROOM-02.P$13, ESP-WROOM-02.P$18, ESP-WROOM-02.P$19, ESP-WROOM-02.P$9, FAN_ON.1, IC1.P$3, IC2.P$7, IC2.P$8, IC2.P$9, JACK.RING, JACK.RING_SW, Q1.S, Q4.2, Q5.2, Q6.2, R14.1, R16.1, R18.1, R5.1, R6.1, R7.1, R8.1, R9.1, RD2.2, REG.1, RT.2, SERIAL4.4, SERIAL6.6, T4.TP; no longer C3.1, C7.P$M, C8.-, ESP1.P$13, ESP1.P$18, ESP1.P$19, ESP1.P$9, ESP2.15, IC2.18, IC2.19, IC2.20, IC2.26, IC2.27, IC2.28, IC3.P$3, IC4.P$3, IC5.3, IC5.4, IC6.P$7, IC6.P$8, IC6.P$9, J2.15, J2.17, J2.18, J2.19, J2.24, J2.3, J2.5, J2.7, Q2.HEAT, Q3.HEAT, R12.1, R14.2, RD2.1, SERIAL.6, U$1.RING, U$1.RING_SW, U1.1
- net HEATER: now also ESP-12.16, ESP-WROOM-02-BREAK.P$6, ESP-WROOM-02.P$6, R15.1, R7.2; no longer R16.1, SJ22.1, SJ5.1
- net HIGH_TEMP: now also ESP-12.4, ESP-WROOM-02-BREAK.P$17, ESP-WROOM-02.P$17, IC1.P$4, R8.2, T7.TP; no longer IC3.P$4, IC4.P$4, R12.2, SJ23.1, SJ8.2
- net N$1: now also RL1.2, RL2.1; no longer J4.1, R10.2
- net N$2: now also HEATER_POWER.2; no longer J3.2
- net N$27: now also IC1.P$2, RH.1; no longer IC3.P$2, IC4.P$2, RH1.1, RH2.1
- net N$3: now also HEATSINK.P$1, Q1.D, RELAY.P$5; no longer Q2.1, R16.2
- net N$4: now also FAN.3, FAN_ON.2; no longer JP2.3
- net N$5: now also Q1.G, Q6.3, R13.1, R14.2; no longer Q3.1, R15.2
- net N$6: now also PEL_RED.1, RELAY.P$8; no longer IC2.6, R5.2
- net N$7: now also PEL_BLK.1, RELAY.P$1; no longer IC2.10, R6.2
- net N$8: now also Q3.1, R17.2, R18.2; no longer IC2.5, R1.2
- net N$92: now also C1.2, IC2.P$6; no longer C3.2, IC6.P$6
- net PEL_PWM: now also ESP-12.19, ESP-WROOM-02-BREAK.P$10, ESP-WROOM-02.P$10, R12.1; no longer R3.1, SJ14.2, SJ28.2
- net RESET: now also ESP-12.1, ESP-WROOM-02-BREAK.P$15, ESP-WROOM-02.P$15, R1.2, T6.TP; no longer R9.2, SJ10.2, SJ15.1
- net RXD: now also ESP-12.21, ESP-WROOM-02-BREAK.P$11, ESP-WROOM-02.P$11, SERIAL4.2, SERIAL6.3, T2.TP; no longer SERIAL.2, SJ13.2, SJ25.2
- net TXD: now also ESP-12.22, ESP-WROOM-02-BREAK.P$12, ESP-WROOM-02.P$12, SERIAL4.3, SERIAL6.2, T1.TP; no longer SERIAL.3, SJ12.2, SJ24.2
- net WELL_TEMP: now also IC2.P$3, RH.2, RL2.2; no longer RH1.2, RH2.2, RL.1, SJ17.2
Routing:
- net PEL_INB: track 151.9 -> 0.00 mm, vias 3 -> 0
- net PEL_SWA: track 0.00 -> 118.2 mm, vias 0 -> 3
- net 12V: track 296.9 -> 183.3 mm, vias 45 -> 0
- net GND: track 701.6 -> 809.8 mm, vias 81 -> 47
- net INT_ADC: track 96.3 -> 0.00 mm, vias 1 -> 0
- net OUTB: track 91.9 -> 0.00 mm, vias 16 -> 0
- net TXD: track 17.1 -> 107.2 mm, vias 1 -> 2
- net FAN: track 28.3 -> 118.4 mm, vias 1 -> 4
- net MODE: track 0.00 -> 89.7 mm, vias 0 -> 4
- net DRDY: track 0.00 -> 89.6 mm, vias 0 -> 4
- net IO2: track 85.7 -> 0.00 mm, vias 2 -> 0
- net RXD: track 15.2 -> 100.7 mm, vias 1 -> 2
- net IO5: track 75.0 -> 0.00 mm, vias 2 -> 0
- net N$3: track 29.9 -> 99.2 mm, vias 0 -> 6
- net SCLK: track 0.00 -> 67.2 mm, vias 0 -> 3
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- removed copper zone on layer 1, net 12V
- removed copper zone on layer 16, net 12V
- removed copper zone on layer 1, net OUTA
- removed copper zone on layer 16, net OUTA
- removed copper zone on layer 16, net OUTB
Other:
- board outline removed
- board text added: "*"
- board text added: "+"
- board text added: "63 x 86 mm"
- board text added: "ATX"
- board text added: "C1"
- board text added: "C2"
- board text added: "C3"
- board text added: "C4"
- board text added: "CP1"
- board text added: "CP2"
- board text added: "D1"
- board text added: "D2"
- board text added: "ESP-12"
- board text added: "HEATER POWER"
- board text added: "HEATER TEMP"
- board text added: "HEATSINK"
- board text added: "IC1"
- board text added: "IC2"
- board text added: "IO0"
- board text added: "MODE"
- board text added: "NinjaPCB-4x4-NinNin ver2.0"
- board text added: "ON"
- board text added: "PEL BLK"
- board text added: "PEL RED"
- board text added: "Q1"
- board text added: "Q4"
- board text added: "Q5"
- board text added: "Q6"
- board text added: "R1"
- board text added: "R10"
- board text added: "R11"
- board text added: "R12"
- board text added: "R13"
- board text added: "R14"
- board text added: "R15"
- board text added: "R16"
- board text added: "R17"
- board text added: "R18"
- board text added: "R2"
- board text added: "R3"
- board text added: "R4"
- board text added: "R5"
- board text added: "R6"
- board text added: "R7"
- board text added: "R8"
- board text added: "R9"
- board text added: "RD1"
- board text added: "RD2"
- board text added: "REG"
- board text added: "RELAY"
- board text added: "RH"
- board text added: "RL1"
- board text added: "RL2"
- board text added: "RST"
- board text added: "RT"
- board text added: "SERIAL4"
- board text added: "SERIAL6"
- board text added: "T1"
- board text added: "T2"
- board text added: "T3"
- board text added: "T4"
- board text added: "T5"
- board text added: "T6"
- board text added: "T7"
- board text added: "https://github.com/hisashin/NinjaPCR"
- board text removed: "BLACK"
- board text removed: "ESP-12F"
- board text removed: "GND"
- board text removed: "HEATER"
- board text removed: "HEATER_TEMP"
- board text removed: "High Precision"
- board text removed: "I2C"
- board text removed: "J1"
- board text removed: "J3"
- board text removed: "J4"
- board text removed: "J5"
- board text removed: "JP2"
- board text removed: "NinjaPCB ver2-170831"
- board text removed: "PELTIER"
- board text removed: "RED"
- board text removed: "RX"
- board text removed: "SPI"
- board text removed: "TX"

Commit message: remove wrong schematics
Parts:
- RELAY: value NEC-RELAY2EP2 -> NEC-RELAY2EN2; device PCR-Switch:NEC-EP2 -> PCR-Switch:NEC-EN2
Changed lines of the file:
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@@
 <setting verticaltext="up"/>
 </settings>
-<grid distance="1" unitdist="mil" unit="mil" style="lines" multiple="1" display="yes" altdistance="0.025" altunitdist="inch" altunit="inch"/>
+<grid distance="1" unitdist="mil" unit="mm" style="lines" multiple="1" display="yes" altdistance="0.025" altunitdist="inch" altunit="inch"/>
 <layers>
 <layer number="1" name="Top" color="4" fill="1" visible="yes" active="yes"/>
@@
 <attribute name="MPN" value="RC0603JR-0710KL" x="-58.674" y="1.524" size="1.778" layer="27" rot="R270" display="off"/>
 </element>
-<element name="RELAY" library="PCR-Switch" package="NEC-EP2" value="NEC-RELAY2EP2" x="20.2176" y="63.7048" smashed="yes" rot="R270"/>
+<element name="RELAY" library="PCR-Switch" package="NEC-EN2" value="NEC-RELAY2EN2" x="20.2176" y="63.7048" smashed="yes" rot="R270"/>
 <element name="D1" library="Seeed-Diode" package="DO-214AC" value="1N4007" x="10.243" y="74.684" smashed="yes" rot="R270">
 <attribute name="MPN" value="1N4007" x="-68.497" y="2.294" size="1.778" layer="27" rot="R270" display="off"/>
