File: eagle/NinjaPCB_ver2.1.sch (EAGLE design)
At the start: 75 parts, among them IC1 ANALOGSW_AD_SOT23-6, IC2 NAU7802, Q1 IRLB3813PBF, Q2 CJ2302, Q3 CJ2302, Q4 S9013, Q5 S9013, Q6 S9013, T1 TPTP20R, T2 TPTP20R, T3 TPTP20R, T4 TPTP20R, T5 TPTP20R, T6 TPTP20R, T7 TPTP20R

Commit message: update dxf
Parts:
- added R20: 0R, Seeed-Resistor:SMD-RES-0R-5%-1/10W(0603)
Connections:
- net GND: now also R20.1
- net N$4: now also R20.2
Other:
- note added: "Diff from ver2.0: 1. ATX:POWER_ON is connected to GND so that ATX works 2. Add R19 in case ESP can drive MOSFET directly. 3. FAN_ON jumper removed. it should be turn off while heating 4. Relay EP2 library was wrongly designed with EN2 specs. Corrected 5. 0ohm added to Fan"
- note removed: "Diff from ver2.0: 1. ATX:POWER_ON is connected to GND so that ATX works 2. Add R19 in case ESP can drive MOSFET directly. 3. FAN_ON jumper removed. it should be turn off while heating 4. Relay EP2 library was wrongly designed with EN2 specs. Corrected"
Changed lines of the file:
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@@
 <setting verticaltext="up"/>
 </settings>
-<grid distance="0.1" unitdist="inch" unit="inch" style="lines" multiple="1" display="no" altdistance="0.01" altunitdist="inch" altunit="inch"/>
+<grid distance="0.05" unitdist="inch" unit="inch" style="lines" multiple="1" display="no" altdistance="0.01" altunitdist="inch" altunit="inch"/>
 <layers>
 <layer number="1" name="Top" color="4" fill="1" visible="no" active="no"/>
@@
 <part name="U$10" library="adafruit" deviceset="FIDUCIAL" device=""/>
 <part name="R19" library="Seeed-Resistor" deviceset="SMD-RES-1K-5%-1/10W(0603)" device="" value="1K 1/10W"/>
+<part name="R20" library="Seeed-Resistor" deviceset="SMD-RES-0R-5%-1/10W(0603)" device="" value="0R"/>
 </parts>
 <sheets>
@@
 <text x="26.67" y="238.76" size="3.81" layer="97">MCU</text>
 <text x="149.86" y="77.47" size="3.81" layer="97">POWER</text>
-<text x="1.27" y="-12.7" size="1.778" layer="97">Diff from ver2.0:
+<text x="1.27" y="-19.05" size="1.778" layer="97">Diff from ver2.0:
 1. ATX:POWER_ON is connected to GND so that ATX works
 2. Add R19 in case ESP can drive MOSFET directly.
 3. FAN_ON jumper removed. it should be turn off while heating
-4. Relay EP2 library was wrongly designed with EN2 specs. Corrected</text>
+4. Relay EP2 library was wrongly designed with EN2 specs. Corrected
+5. 0ohm added to Fan</text>
 <text x="22.86" y="129.54" size="3.81" layer="97">CONFIG</text>
 <text x="86.36" y="-22.86" size="1.778" layer="97">Notes for wiring:
@@
 <instance part="U$10" gate="G$1" x="135.89" y="21.59"/>
 <instance part="R19" gate="G$1" x="293.37" y="179.07"/>
+<instance part="R20" gate="G$1" x="337.82" y="55.88" rot="R90"/>
 </instances>
 <busses>
@@
 <wire x1="327.66" y1="49.53" x2="330.2" y2="49.53" width="0.1524" layer="91"/>
 <junction x="330.2" y="49.53"/>
+<pinref part="R20" gate="G$1" pin="1"/>
+<wire x1="330.2" y1="49.53" x2="337.82" y2="49.53" width="0.1524" layer="91"/>
+<wire x1="337.82" y1="49.53" x2="337.82" y2="52.07" width="0.1524" layer="91"/>
 </segment>
 <segment>
@@
 <net name="N$4" class="0">
 <segment>
-<wire x1="340.36" y1="63.5" x2="330.2" y2="63.5" width="0.1524" layer="91"/>
+<wire x1="340.36" y1="63.5" x2="337.82" y2="63.5" width="0.1524" layer="91"/>
+<wire x1="337.82" y1="63.5" x2="330.2" y2="63.5" width="0.1524" layer="91"/>
 <wire x1="330.2" y1="63.5" x2="330.2" y2="62.23" width="0.1524" layer="91"/>
 <pinref part="FAN" gate="-3" pin="S"/>
 <pinref part="Q3" gate="G$1" pin="D"/>
+<pinref part="R20" gate="G$1" pin="2"/>
+<wire x1="337.82" y1="59.69" x2="337.82" y2="63.5" width="0.1524" layer="91"/>
+<junction x="337.82" y="63.5"/>
 </segment>
 </net>

Commit message: ver2.1 finished
Parts:
- removed PEL_BLK, PEL_RED: (no value), pinhead:PINHD-1X1L
- removed T1, T2, T3, T4, T5, T6, T7: TPTP20R, testpad:TPTP20R
- removed U$6: FIDUCIAL, adafruit:FIDUCIAL
- added DIN4: DIN4, PCR-Connector:DIN4
- added PELTIER: (no value), Seeed-Connector:SCREW-TERMINAL-GREEN(2P-3.5)
- added R21: 0R, Seeed-Resistor:SMD-RES-0R-5%-1/10W(0603)
- added RESET: (no value), pinhead:PINHD-1X2
- IO0: device Seeed-Switch:DIP-SWITCH-TACTILE-SPST-NO/TS-1109(4P-D6.0MM)'TS-1109' -> pinhead:PINHD-1X2
- R12, R15: value 1K 1/10W -> 10K 1/10W; device Seeed-Resistor:SMD-RES-1K-5%-1/10W(0603) -> Seeed-Resistor:SMD-RES-10K-5%-1/10W(0603)
- R13, R14: value 10K 1/10W -> 1K 1/10W; device Seeed-Resistor:SMD-RES-10K-5%-1/10W(0603) -> Seeed-Resistor:SMD-RES-1K-5%-1/10W(0603)
- R20: value 0R -> 10K 1/10W; device Seeed-Resistor:SMD-RES-0R-5%-1/10W(0603) -> Seeed-Resistor:SMD-RES-10K-5%-1/10W(0603)
- WELL_TEMP: device pinhead:PINHD-1X2 -> pinhead:PINHD-1X2/90
Connections:
- removed net N$6: PEL_RED.1, RELAY.8
- removed net N$7: PEL_BLK.1, RELAY.1
- new net BLK: PELTIER.2, RELAY.1
- new net RED: PELTIER.1, RELAY.8
- net 12V: now also DIN4.P$1, DIN4.P$2, R15.2; no longer R13.2
- net 3V3: now also R9.2; no longer T3.TP
- net FAN: now also IO0.1, R19.1; no longer IO0.A0, IO0.A1, R17.1, T5.TP
- net GND: now also DIN4.P$3, DIN4.P$4, DIN4.P$6, DIN4.P$7, DIN4.P$8, DIN4.P$9, IO0.2, R10.2, R21.1; no longer IO0.B0, IO0.B1, R14.1, R9.1, T4.TP
- net HEATER: now also R17.1; no longer R15.1
- net HIGH_TEMP: now also RESET.2; no longer T7.TP
- net MODE: now also R10.1, R9.1; no longer R9.2
- net N$30: now also R13.2, R14.1; no longer R12.2, R19.1
- net N$32: now also R17.2, R18.2; no longer R15.2, R16.2
- net N$34: now also R11.2; no longer R10.2
- net N$35: now also R12.1; no longer R11.1
- net N$4: now also R21.2; no longer R20.2
- net N$5: now also R15.1, R16.2; no longer R13.1, R19.2
- net N$8: now also R19.2, R20.2; no longer R17.2, R18.2
- net PEL_PWM: now also R13.1; no longer R12.1
- net PEL_SWA: now also R11.1; no longer R10.1
- net PEL_SWB: now also R12.2; no longer R11.2
- net RESET: now also RESET.1; no longer T6.TP
- net RXD: no longer T2.TP
- net TXD: no longer T1.TP
Other:
- note added: "Diff from ver2.0: 1. ATX:POWER_ON is connected to GND so that ATX works 2. Add R19 in case ESP can drive MOSFET directly. 3. FAN_ON jumper removed. it should be turn off while heating 4. Relay EP2 library was wrongly designed with EN2 specs. Corrected 5. 0ohm added to Fan 6. Peltier is connected to terminal block (must be bigger?) 7. DIN4 power added 8. IO0 tact is replaced with simple jumper 9. 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"
- note removed: "Diff from ver2.0: 1. ATX:POWER_ON is connected to GND so that ATX works 2. Add R19 in case ESP can drive MOSFET directly. 3. FAN_ON jumper removed. it should be turn off while heating 4. Relay EP2 library was wrongly designed with EN2 specs. Corrected 5. 0ohm added to Fan"
- moved on the sheet: ATX, C1, C2, C3, C4, ESP-WROOM-02-BREAK, HEATER_TEMP, IC1, IC2, JACK, MODE, R1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

Commit message: minor update of silk
Parts:
- RT: value 5K HP -> 4.99K HP
- renumbered ESP-12 to ESP1, ESP-WROOM-02 to ESP2, ESP-WROOM-02-BREAK to ESP3
