File: eagle/NinjaPCB_ver2.2.sch (EAGLE design)
At the start: 72 parts, among them IC1 ANALOGSW_AD_SOT23-5, IC2 NAU7802, Q1 IRLB3813PBF, Q2 CJ2302, Q3 CJ2302, Q4 S9013, Q5 S9013, Q6 S9013

Commit message: updated 2.2
Parts:
- R9: value 10K 1/10W -> 100K 1/10W; device Seeed-Resistor:SMD-RES-10K-5%-1/10W(0603) -> Seeed-Resistor:SMD-RES-100K-5%-1/10W(0603)
Other:
- note added: "KEEP R9, R14 and R21 OPEN"
Changed lines of the file:
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@@
 <part name="GND17" library="supply1" deviceset="GND" device=""/>
 <part name="IO0" library="pinhead" deviceset="PINHD-1X2" device=""/>
-<part name="R9" library="Seeed-Resistor" deviceset="SMD-RES-10K-5%-1/10W(0603)" device="" value="10K 1/10W"/>
+<part name="R9" library="Seeed-Resistor" deviceset="SMD-RES-100K-5%-1/10W(0603)" device="" value="100K 1/10W"/>
 <part name="3V12" library="supply1" deviceset="VCC" device="" value="3V3"/>
 <part name="GND19" library="supply1" deviceset="GND" device=""/>
@@
 <text x="26.67" y="238.76" size="3.81" layer="97">MCU</text>
 <text x="148.59" y="92.71" size="3.81" layer="97">POWER</text>
-<text x="1.27" y="-13.97" size="1.778" layer="97">Diff from ver2.1:
+<text x="255.27" y="8.89" size="1.778" layer="97">Diff from ver2.1:
 1. Serial doesn't power
 2. Rename MODE to TOUT
@@
 4. Stable EN</text>
 <text x="19.05" y="92.71" size="3.81" layer="97">CONFIG</text>
+<text x="6.35" y="247.65" size="6.4516" layer="97">KEEP R9, R14 and R21 OPEN</text>
 </plain>
 <instances>
