File: eagle/NinjaPCB_ver2.2.brd (EAGLE design)
At the start: 79 x 73 mm, 72 parts, among them IC1 ANALOGSW_AD_SOT23-6, IC2 NAU7802, Q1 IRLB3813PBF, Q2 CJ2302, Q3 CJ2302, Q4 S9013, Q5 S9013, Q6 S9013

Commit message: NinjaPCB ver2.2
Parts:
- removed U$6: (no value), oshw:OSHW_16MM
- added U$2: (no value), oshw:OSHW_5MM
- moved R1 61.1 mm to (48.0, 61.6), turned to 90 degrees
- moved R8 54.1 mm to (48.0, 55.0), turned to 90 degrees
- moved R5 2.54 mm to (48.0, 52.8)
- moved R6 2.18 mm to (48.0, 50.6)
- moved R7 1.83 mm to (48.0, 48.5)
- moved R9 1.07 mm to (48.0, 59.4)
- moved R4 0.76 mm to (48.0, 63.8)
- moved R10 0.71 mm to (48.0, 57.2)
- moved R3 0.41 mm to (48.0, 65.9)
- moved R2 0.05 mm to (48.0, 68.1)
Connections:
- net 3V3: no longer SERIAL4.1, SERIAL6.4
Routing:
- net GND: track 918.2 -> 878.0 mm, vias 50 -> 47
- net 3V3: track 247.2 -> 214.1 mm
- net RESET: track 107.6 -> 131.0 mm, vias 2 -> 3
- net HIGH_TEMP: track 128.2 -> 140.0 mm, vias 3 -> 4
- net TXD: track 88.3 -> 96.7 mm
- net PEL_SWA: track 143.0 -> 148.8 mm
- net MODE: track 95.0 -> 98.3 mm
- net RXD: track 85.0 -> 87.3 mm
- net HEATER: track 78.7 -> 80.5 mm
- net SCLK: track 79.3 -> 80.1 mm
Other:
- board text added: "NinjaPCB"
- board text added: "NinjaPCB ver2.2"
- board text added: "^R14*"
- board text added: "^R21"
- board text added: "^R9"
- board text removed: "NinjaPCB ver2.1"
- board text removed: "R14*"
- board text removed: "R21"
- board text removed: "R9"
- board text removed: "https://github.com/hisashin/NinjaPCR"

Commit message: fixed NinjaPCB ver 2.2
Parts:
- added C5: 100nf, Seeed-Capacitor:C0603
- added R22: 1K 1/10W, Seeed-Resistor:R0603
- IC1: value ANALOGSW_AD_SOT23-6 -> ANALOGSW_AD_SOT23-5; device PCR-IC:SOT-23-6 -> PCR-IC:SOT23-5
- R14: value 1K 1/10W -> 0R
- turned IC1 to 270 degrees
Connections:
- net MODE renamed TOUT
- net 3V3: now also IC1.1, IC1.6, R22.2; no longer IC1.P$1, IC1.P$6
- net EN: now also C5.2, R22.1
- net GND: now also C5.1, IC1.3; no longer IC1.P$3
- net HIGH_TEMP: now also IC1.4; no longer IC1.P$4
- net N$27: now also IC1.2; no longer IC1.P$2
Routing:
- net 3V3: track 214.1 -> 219.5 mm
- net EN: track 50.3 -> 54.5 mm
- net GND: track 878.0 -> 874.3 mm
- net TOUT: track 98.3 -> 97.7 mm
- net RESET: track 131.0 -> 130.5 mm
Other:
- board text added: "C5"
- board text added: "R22"
- board text added: "^R14"
- board text removed: "^R14*"

Commit message: updated 2.2
Parts:
- R9: value 10K 1/10W -> 100K 1/10W
Other:
- board text added: "R22*"
- board text removed: "R22"
Changed lines of the file:
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@@
 <text x="28.0416" y="45.8216" size="1.27" layer="21" font="vector" rot="R180">C1</text>
 <text x="25.3492" y="52.6288" size="1.27" layer="21" font="vector" rot="R180">C2</text>
-<text x="41.5798" y="47.4472" size="1.27" layer="21" font="vector">IC1</text>
+<text x="40.0812" y="46.9646" size="1.27" layer="21" font="vector" rot="R180">IC1</text>
 <text x="31.5468" y="50.1396" size="1.27" layer="21" font="vector">IC2</text>
 <text x="38.5572" y="66.8782" size="1.27" layer="21" font="vector">WELL
@@
 <text x="4.2418" y="60.96" size="1.27" layer="21" font="vector" rot="R180">Q3</text>
 <text x="4.2418" y="63.5" size="1.27" layer="21" font="vector" rot="R180">R20</text>
-<text x="4.2418" y="66.04" size="1.016" layer="21" font="vector" rot="R180">R19*</text>
+<text x="4.2672" y="65.4558" size="1.016" layer="21" font="vector" rot="R180">R19*</text>
 <text x="12.5476" y="62.0522" size="1.27" layer="21" font="vector" rot="R180">FAN</text>
 <text x="26.9494" y="57.8104" size="1.27" layer="21" font="vector" rot="R180">Q2</text>
@@
 <text x="46.7614" y="62.23" size="1.27" layer="21" font="vector" rot="R180">R1</text>
 <text x="46.7614" y="55.6768" size="1.27" layer="21" font="vector" rot="R180">R8</text>
-<text x="51.2318" y="61.214" size="1.27" layer="21" font="vector" rot="R90">R22</text>
+<text x="51.2318" y="61.214" size="1.016" layer="21" font="vector" rot="R90">R22*</text>
 <text x="51.2318" y="57.277" size="1.27" layer="21" font="vector" rot="R90">C5</text>
 </plain>
@@
 <attribute name="VALUE" x="57.7342" y="10.0076" size="1.27" layer="28" rot="MR0"/>
 </element>
-<element name="R9" library="Seeed-Resistor" package="R0603" value="10K 1/10W" x="48.006" y="59.3852" smashed="yes" rot="R270">
-<attribute name="MPN" value="RC0603JR-0710KL" x="48.006" y="59.3852" size="1.778" layer="27" rot="R270" display="off"/>
+<element name="R9" library="Seeed-Resistor" package="R0603" value="100K 1/10W" x="48.006" y="59.3852" smashed="yes" rot="R270">
+<attribute name="MPN" value="RC0603JR-07100KL" x="48.006" y="59.3852" size="1.778" layer="27" rot="R270" display="off"/>
 </element>
 <element name="RESET" library="pinhead" package="1X02" value="" x="60.2742" y="13.1826" smashed="yes" rot="MR0">
@@
 <attribute name="NAME" x="52.2986" y="57.4548" size="0.635" layer="33" ratio="10" rot="R90"/>
 </element>
-<element name="IC1" library="PCR-IC" package="SOT23-5" value="ANALOGSW_AD_SOT23-5" x="39.8842" y="49.0394" rot="R270"/>
+<element name="IC1" library="PCR-IC" package="SOT23-5" value="ANALOGSW_AD_SOT23-5" x="39.8842" y="49.0394" smashed="yes" rot="R270"/>
 </elements>
 <signals>
@@
 <wire x1="38.8366" y1="53.0606" x2="40.005" y2="53.0606" width="0.4064" layer="16"/>
 <via x="37.338" y="51.8414" extent="1-16" drill="0.6" shape="square"/>
-<wire x1="38.1256" y1="50.1394" x2="37.338" y2="50.927" width="0.4064" layer="1"/>
-<wire x1="37.338" y1="50.927" x2="37.338" y2="51.8414" width="0.4064" layer="1"/>
+<wire x1="37.338" y1="50.927" x2="37.338" y2="51.3334" width="0.4064" layer="1"/>
+<wire x1="37.338" y1="51.3334" x2="37.338" y2="51.8414" width="0.4064" layer="1"/>
 <wire x1="34.036" y1="68.072" x2="34.2646" y2="68.072" width="0.4064" layer="1"/>
 <wire x1="34.2646" y1="68.072" x2="36.322" y2="66.0146" width="0.4064" layer="1"/>
@@
 <wire x1="52.1208" y1="57.8866" x2="52.1208" y2="55.9308" width="0.4064" layer="1"/>
 <contactref element="IC1" pad="3"/>
-<wire x1="51.7398" y1="29.4386" x2="56.7436" y2="25.2984" width="0" layer="19" extent="1-1"/>
-<wire x1="71.7804" y1="3.2004" x2="77.159" y2="6.817" width="0" layer="19" extent="1-1"/>
-<wire x1="61.7982" y1="5.8674" x2="67.6656" y2="11.1252" width="0" layer="19" extent="1-1"/>
-<wire x1="38.1256" y1="50.1394" x2="38.9342" y2="50.1394" width="0.4064" layer="1"/>
-<wire x1="38.9342" y1="50.1394" x2="38.9342" y2="50.2332" width="0.4064" layer="1"/>
+<wire x1="38.9342" y1="50.2332" x2="37.8286" y2="50.2332" width="0.4064" layer="1"/>
+<wire x1="37.8286" y1="50.2332" x2="37.338" y2="50.7238" width="0.4064" layer="1"/>
+<wire x1="37.338" y1="50.7238" x2="37.338" y2="50.927" width="0.4064" layer="1"/>
 </signal>
 <signal name="3V3">
@@
 <contactref element="IC1" pad="6"/>
 <wire x1="40.8342" y1="51.0376" x2="40.8342" y2="50.2332" width="0.4064" layer="1"/>
-<wire x1="40.8342" y1="50.2332" x2="40.8342" y2="47.8456" width="0.4064" layer="1"/>
+<wire x1="40.8342" y1="47.8456" x2="40.8342" y2="50.2332" width="0.4064" layer="1"/>
 <wire x1="40.7924" y1="46.6598" x2="40.8342" y2="46.6598" width="0.4064" layer="1"/>
 <wire x1="40.8342" y1="46.6598" x2="40.8342" y2="47.8456" width="0.4064" layer="1"/>
@@
 <wire x1="49.7078" y1="54.0512" x2="50.0126" y2="54.0512" width="0.4064" layer="1"/>
 <contactref element="IC1" pad="4"/>
-<wire x1="38.9342" y1="46.8416" x2="38.9342" y2="47.8456" width="0.4064" layer="1"/>
+<wire x1="38.9342" y1="47.8456" x2="38.9342" y2="46.8416" width="0.4064" layer="1"/>
 </signal>
 <signal name="N$92">
@@
 <wire x1="35.6616" y1="55.2196" x2="39.8842" y2="50.997" width="0.4064" layer="1"/>
 <contactref element="IC1" pad="2"/>
-<wire x1="39.8842" y1="50.997" x2="39.8842" y2="50.2332" width="0.4064" layer="1"/>
+<wire x1="39.8842" y1="50.2332" x2="39.8842" y2="50.997" width="0.4064" layer="1"/>
 </signal>
 <signal name="WELL_TEMP">
