File: eagle/breakout/ESP-12F-ASIF-WR02.brd (EAGLE design)
At the start: 29 x 24 mm, 10 parts

Commit message: latest updates
Other:
- board text added: "ESP-12F-ASIF-WR02"
- board text removed: "ESP-12F-BREAK"
Changed lines of the file:
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@@
 <text x="3.302" y="-8.382" size="1.016" layer="22" font="vector" rot="MR90">MOSI</text>
 <text x="5.842" y="-8.382" size="1.016" layer="22" font="vector" rot="MR90">SCLK</text>
-<text x="-5.8674" y="11.6586" size="1.016" layer="22" font="vector" rot="MR180">ESP-12F-BREAK</text>
+<text x="-7.8486" y="11.7856" size="1.016" layer="22" font="vector" rot="MR180">ESP-12F-ASIF-WR02</text>
 </plain>
 <attributes>
