File: eagle/breakout/ESP-WROOM-02-ASIF-12.sch (EAGLE design)
At the start: 9 parts

Commit message: latest updates
Parts:
- LEFT, RIGHT: device pinhead:PINHD-1X9 -> pinhead:PINHD-1X11OCT
- renumbered IO0-3V3 to IO0-PUP, IO0-GND to IO0-PDN, IO15-GND to IO15-PDN, IO2-3V3 to IO2-PUP, U$1 to U1
Connections:
- new net NC1: LEFT.9
- new net NC2: LEFT.10
- new net NC3: LEFT.11
- new net NC4: RIGHT.11
- new net NC5: RIGHT.10
- new net NC6: RIGHT.9
- net 3V3: now also LEFT.8; no longer LEFT.1
- net EN: now also LEFT.3; no longer LEFT.2
- net GND: now also RIGHT.8; no longer LEFT.9, RIGHT.1, RIGHT.6
- net IO0: now also RIGHT.5; no longer LEFT.8
- net IO12: now also LEFT.6; no longer LEFT.4
- net IO13: now also LEFT.7; no longer LEFT.5
- net IO14: now also LEFT.5; no longer LEFT.3
- net IO15: now also RIGHT.7; no longer LEFT.6
- net IO16: now also LEFT.4; no longer RIGHT.2
- net IO2: now also RIGHT.6; no longer LEFT.7
- net IO4: now also RIGHT.4; no longer RIGHT.9
- net IO5: now also RIGHT.3; no longer RIGHT.5
- net RST: now also LEFT.1; no longer RIGHT.4
- net RXD: now also RIGHT.2; no longer RIGHT.8
- net TOUT: now also LEFT.2; no longer RIGHT.3
- net TXD: now also RIGHT.1; no longer RIGHT.7
