File: eagle/breakout/writer2.brd (EAGLE design)
At the start: 40 x 20 mm, 3 parts

Commit message: updated 2.2
Parts:
- removed JP3: (no value), pinhead:1X10
Connections:
- net N$1: no longer JP3.10
- net N$10: no longer JP3.1
- net N$2: no longer JP3.9
- net N$3: no longer JP3.8
- net N$4: no longer JP3.7
- net N$5: no longer JP3.6
- net N$6: no longer JP3.5
- net N$7: no longer JP3.4
- net N$8: no longer JP3.3
- net N$9: no longer JP3.2
Routing:
- net N$9: track 15.0 -> 7.50 mm
- net N$8: track 15.0 -> 7.50 mm
- net N$7: track 15.0 -> 7.50 mm
- net N$6: track 15.0 -> 7.50 mm
- net N$5: track 15.0 -> 7.50 mm
- net N$4: track 15.0 -> 7.50 mm
- net N$3: track 15.0 -> 7.50 mm
- net N$2: track 15.0 -> 7.50 mm
- net N$10: track 15.0 -> 7.50 mm
- net N$1: track 15.0 -> 7.50 mm
Changed lines of the file:
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@@
 <attribute name="VALUE" x="-12.7" y="-10.675" size="1.27" layer="27"/>
-</element>
-<element name="JP3" library="pinhead" package="1X10" value="" x="0" y="7.5" smashed="yes">
-<attribute name="VALUE" x="-12.7" y="4.325" size="1.27" layer="27"/>
 </element>
 </elements>
@@
 <contactref element="JP2" pad="10"/>
 <wire x1="11.43" y1="0" x2="11.43" y2="-7.5" width="1.27" layer="16"/>
-<contactref element="JP3" pad="10"/>
-<wire x1="11.43" y1="7.5" x2="11.43" y2="0" width="1.27" layer="1"/>
 </signal>
 <signal name="N$2">
@@
 <contactref element="JP2" pad="9"/>
 <wire x1="8.89" y1="0" x2="8.89" y2="-7.5" width="1.27" layer="16"/>
-<contactref element="JP3" pad="9"/>
-<wire x1="8.89" y1="7.5" x2="8.89" y2="0" width="1.27" layer="1"/>
 </signal>
 <signal name="N$3">
@@
 <contactref element="JP2" pad="8"/>
 <wire x1="6.35" y1="0" x2="6.35" y2="-7.5" width="1.27" layer="16"/>
-<contactref element="JP3" pad="8"/>
-<wire x1="6.35" y1="7.5" x2="6.35" y2="0" width="1.27" layer="1"/>
 </signal>
 <signal name="N$4">
@@
 <contactref element="JP2" pad="7"/>
 <wire x1="3.81" y1="0" x2="3.81" y2="-7.5" width="1.27" layer="16"/>
-<contactref element="JP3" pad="7"/>
-<wire x1="3.81" y1="7.5" x2="3.81" y2="0" width="1.27" layer="1"/>
 </signal>
 <signal name="N$5">
@@
 <contactref element="JP2" pad="6"/>
 <wire x1="1.27" y1="0" x2="1.27" y2="-7.5" width="1.27" layer="16"/>
-<contactref element="JP3" pad="6"/>
-<wire x1="1.27" y1="7.5" x2="1.27" y2="0" width="1.27" layer="1"/>
 </signal>
 <signal name="N$6">
@@
 <contactref element="JP2" pad="5"/>
 <wire x1="-1.27" y1="0" x2="-1.27" y2="-7.5" width="1.27" layer="16"/>
-<contactref element="JP3" pad="5"/>
-<wire x1="-1.27" y1="7.5" x2="-1.27" y2="0" width="1.27" layer="1"/>
 </signal>
 <signal name="N$7">
@@
 <contactref element="JP2" pad="4"/>
 <wire x1="-3.81" y1="0" x2="-3.81" y2="-7.5" width="1.27" layer="16"/>
-<contactref element="JP3" pad="4"/>
-<wire x1="-3.81" y1="7.5" x2="-3.81" y2="0" width="1.27" layer="1"/>
 </signal>
 <signal name="N$8">
@@
 <contactref element="JP2" pad="3"/>
 <wire x1="-6.35" y1="0" x2="-6.35" y2="-7.5" width="1.27" layer="16"/>
-<contactref element="JP3" pad="3"/>
-<wire x1="-6.35" y1="7.5" x2="-6.35" y2="0" width="1.27" layer="1"/>
 </signal>
 <signal name="N$9">
@@
 <contactref element="JP2" pad="2"/>
 <wire x1="-8.89" y1="0" x2="-8.89" y2="-7.5" width="1.27" layer="16"/>
-<contactref element="JP3" pad="2"/>
-<wire x1="-8.89" y1="7.5" x2="-8.89" y2="0" width="1.27" layer="1"/>
 </signal>
 <signal name="N$10">
@@
 <contactref element="JP2" pad="1"/>
 <wire x1="-11.43" y1="0" x2="-11.43" y2="-7.5" width="1.27" layer="16"/>
-<contactref element="JP3" pad="1"/>
-<wire x1="-11.43" y1="7.5" x2="-11.43" y2="0" width="1.27" layer="1"/>
 </signal>
 </signals>
