File: eagle/breakout/writer2.sch (EAGLE design)
At the start: 3 parts

Commit message: updated 2.2
Parts:
- removed JP3: (no value), pinhead:PINHD-1X10
Connections:
- net N$1: no longer JP3.10
- net N$10: no longer JP3.1
- net N$2: no longer JP3.9
- net N$3: no longer JP3.8
- net N$4: no longer JP3.7
- net N$5: no longer JP3.6
- net N$6: no longer JP3.5
- net N$7: no longer JP3.4
- net N$8: no longer JP3.3
- net N$9: no longer JP3.2
Changed lines of the file:
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@@
 <part name="JP1" library="pinhead" deviceset="PINHD-1X10" device=""/>
 <part name="JP2" library="pinhead" deviceset="PINHD-1X10" device=""/>
-<part name="JP3" library="pinhead" deviceset="PINHD-1X10" device=""/>
 </parts>
 <sheets>
@@
 <instance part="JP1" gate="A" x="2.54" y="17.78" rot="MR0"/>
 <instance part="JP2" gate="A" x="17.78" y="17.78"/>
-<instance part="JP3" gate="A" x="27.94" y="17.78"/>
 </instances>
 <busses>
@@
 <pinref part="JP2" gate="A" pin="10"/>
 <wire x1="5.08" y1="5.08" x2="15.24" y2="5.08" width="0.1524" layer="91"/>
-<pinref part="JP3" gate="A" pin="10"/>
-<wire x1="25.4" y1="5.08" x2="15.24" y2="5.08" width="0.1524" layer="91"/>
 </segment>
 </net>
@@
 <pinref part="JP2" gate="A" pin="9"/>
 <wire x1="5.08" y1="7.62" x2="15.24" y2="7.62" width="0.1524" layer="91"/>
-<pinref part="JP3" gate="A" pin="9"/>
-<wire x1="25.4" y1="7.62" x2="15.24" y2="7.62" width="0.1524" layer="91"/>
 </segment>
 </net>
@@
 <pinref part="JP2" gate="A" pin="8"/>
 <wire x1="5.08" y1="10.16" x2="15.24" y2="10.16" width="0.1524" layer="91"/>
-<pinref part="JP3" gate="A" pin="8"/>
-<wire x1="25.4" y1="10.16" x2="15.24" y2="10.16" width="0.1524" layer="91"/>
 </segment>
 </net>
@@
 <pinref part="JP2" gate="A" pin="7"/>
 <wire x1="5.08" y1="12.7" x2="15.24" y2="12.7" width="0.1524" layer="91"/>
-<pinref part="JP3" gate="A" pin="7"/>
-<wire x1="25.4" y1="12.7" x2="15.24" y2="12.7" width="0.1524" layer="91"/>
 </segment>
 </net>
@@
 <pinref part="JP2" gate="A" pin="6"/>
 <wire x1="5.08" y1="15.24" x2="15.24" y2="15.24" width="0.1524" layer="91"/>
-<pinref part="JP3" gate="A" pin="6"/>
-<wire x1="25.4" y1="15.24" x2="15.24" y2="15.24" width="0.1524" layer="91"/>
 </segment>
 </net>
@@
 <pinref part="JP2" gate="A" pin="5"/>
 <wire x1="5.08" y1="17.78" x2="15.24" y2="17.78" width="0.1524" layer="91"/>
-<pinref part="JP3" gate="A" pin="5"/>
-<wire x1="25.4" y1="17.78" x2="15.24" y2="17.78" width="0.1524" layer="91"/>
 </segment>
 </net>
@@
 <pinref part="JP2" gate="A" pin="4"/>
 <wire x1="5.08" y1="20.32" x2="15.24" y2="20.32" width="0.1524" layer="91"/>
-<pinref part="JP3" gate="A" pin="4"/>
-<wire x1="25.4" y1="20.32" x2="15.24" y2="20.32" width="0.1524" layer="91"/>
 </segment>
 </net>
@@
 <pinref part="JP2" gate="A" pin="3"/>
 <wire x1="5.08" y1="22.86" x2="15.24" y2="22.86" width="0.1524" layer="91"/>
-<pinref part="JP3" gate="A" pin="3"/>
-<wire x1="25.4" y1="22.86" x2="15.24" y2="22.86" width="0.1524" layer="91"/>
 </segment>
 </net>
@@
 <pinref part="JP2" gate="A" pin="2"/>
 <wire x1="5.08" y1="25.4" x2="15.24" y2="25.4" width="0.1524" layer="91"/>
-<pinref part="JP3" gate="A" pin="2"/>
-<wire x1="25.4" y1="25.4" x2="15.24" y2="25.4" width="0.1524" layer="91"/>
 </segment>
 </net>
@@
 <pinref part="JP2" gate="A" pin="1"/>
 <wire x1="5.08" y1="27.94" x2="15.24" y2="27.94" width="0.1524" layer="91"/>
-<pinref part="JP3" gate="A" pin="1"/>
-<wire x1="25.4" y1="27.94" x2="15.24" y2="27.94" width="0.1524" layer="91"/>
 </segment>
 </net>
