File: kicad/NinjaPCR/NinjaPCB_ver2.3.sch (KiCad schematic (older format))
At the start: 73 parts, among them IC1 ANALOGSW_AD_SOT23-5, IC2 NAU7802, Q1 IRLB3813PBF, Q2 CJ2302, Q3 CJ2302, Q4 S9013, Q5 S9013, Q6 S9013

Commit message: add link
Parts:
- U1: renamed from U?; footprint RELAY_ACTP_1C8_PAN -> NinjaPCR:ACTP212
Other:
- note added: "Use Panasonic Electric Works ACTP212 instead of EP2 if you cannot get it : https://www.digikey.jp/product-detail/ja/panasonic-electric-works/ACTP212/255-5876-ND/4756498"
Changed lines of the file:
@@
 KEEP R9, R14 and R21 OPEN
 $Comp
-L NinjaPCR:ACTP212 U?
+L NinjaPCR:ACTP212 U1
 U 1 1 607DD8D8
 P 14750 1200
-F 0 "U?" H 15450 500 60  0000 C CNN
+F 0 "U1" H 15450 500 60  0000 C CNN
 F 1 "ACTP212" H 15600 400 60  0000 C CNN
-F 2 "RELAY_ACTP_1C8_PAN" H 15700 450 60  0001 C CNN
+F 2 "NinjaPCR:ACTP212" H 15700 450 60  0001 C CNN
 F 3 "" H 16650 950 60  0000 C CNN
 	1    14750 1200
@@
 $EndComp
 $Comp
-L NinjaPCB_ver2.2-eagle-import:VCC #P+?
+L NinjaPCB_ver2.2-eagle-import:VCC #P+0101
 U 1 1 607DFAF8
 P 15050 750
-F 0 "#P+?" H 15050 750 50  0001 C CNN
+F 0 "#P+0101" H 15050 750 50  0001 C CNN
 F 1 "12V" V 14950 650 59  0000 L BNN
 F 2 "" H 15050 750 50  0001 C CNN
@@
 Wire Wire Line
 	15050 1900 15050 2000
+Text Notes 9200 650  0    50   ~ 0
+Use Panasonic Electric Works ACTP212 instead of EP2 if you cannot get it : https://www.digikey.jp/product-detail/ja/panasonic-electric-works/ACTP212/255-5876-ND/4756498
 $EndSCHEMATC
